File: project_files/W1209_upgrade.sch (KiCad schematic (older format))
At the start: 34 parts, among them J1 Screw_Terminal_01x04, J2 SWIM, J3 PROBE, K1 SANYOU_SRD_Form_C, Q1 S8050, SW1 +, SW2 -, SW3 SET, U1 AMS1117, U2 CA56-12SEKWA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

Commit message: Update W1209_upgrade.sch
Other:
- note added: "If using 10K thermistor:\n- Solder capacitor, use 20K pull-up resistor \n\nIf using DS18B20:\n- Use 4K7 as pull-up resistor instead of 20K\n- DON'T solder capacitor\n\nIf using TMP36 / LM75 / LM335:\n- Replace 0-Ohm resistor with current limiting according to sensor specification\n- Capacitor is optional\n- DON'T solder pull-up resistor"
- note removed: "If using 10K thermistor:\n- Solder capacitor, use 20K pull-up resistor \nIf using DS18B20:\n- Use 4K7 as pull-up resistor instead of 20K\n- DON'T solder capacitor\nIf using TMP36 / LM75 / LM335:\n- Replace 0-Ohm resistor with current limiting according to sensor specification\n- Capacitor is optional\n- DON'T solder pull-up resistor"
- moved on the sheet: C6, D2, D3, J3, K1, Q1, R2, R3, R4, R8, R9
