File: project_files/W1209_upgrade.kicad_pcb (KiCad board)
At the start: 2 copper layers, 49 x 40 mm, 34 parts, among them J1 Screw_Terminal_01x04, J2 SWIM, J3 PROBE, K1 SANYOU_SRD_Form_C, Q1 S8050, SW1 +, SW2 -, SW3 SET, U1 AMS1117, U2 CA56-12SEKWA, U3 STM8S003F3P

Commit message: Comments correction
Parts:
- J1: value Screw_Terminal_01x04 -> SCREWS
- K1: value SANYOU_SRD_Form_C -> SRA-12VDC-AL
- U1: value AMS1117 -> AMS1117-5.0
- renumbered C7 to C5, C5 to C6, C6 to C7, H4 to H1, H3 to H2, H2 to H3, H1 to H4, J3 to J2, J2 to J3, R3 to R2, R4 to R3, R2 to R4, R8 to R7, R7 to R8, SW3 to SW2, SW2 to SW3, U3 to U2, U2 to U3
Connections:
- J2 pad 1: Net-(J3-Pad1) -> +5V
- K1 pad 4: Net-(K1-Pad4) -> unconnected-(K1-Pad4)
- U3 pad 6: Net-(U2-Pad6) -> unconnected-(U3-Pad6)
Other:
- net class Default removed
