File: project_files/W1209_upgrade.kicad_sch (KiCad schematic)
At the start: 33 parts, among them J1 SCREWS, J2 PROBE, J3 SWIM, K1 SRA-12VDC-AL, Q1 S8050, SW1 +, SW2 SET, SW3 -, U1 AMS1117-5.0, U2 STM8S003F3P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

Commit message: updated to KiCAD 10
Parts:
- removed U3: CA56-12SEKWA, Display_7Segment:CA56-12SEKWA, symbol Display_Character:CA56-12SEKWA
- added U4: 2381AS, Display_Segmented:2381, symbol display:2381AS
- C1: footprint Capacitor_THT:CP_Radial_D10.0mm_P2.50mm_P5.00mm -> Capacitor_Tantalum_SMD:CP_EIA-3528-12_Kemet-T_HandSolder
- C7, R7: now not fitted
- H1, H2, H3, H4: footprint MountingHole:MountingHole_3.2mm_M3_ISO14580 -> MountingHole:MountingHole_3.2mm_M3_ISO14580_Pad; symbol Mechanical:MountingHole -> Mechanical:MountingHole_Pad; now left out of the parts list
- J1: footprint TerminalBlock_Phoenix:TerminalBlock_Phoenix_PT-1,5-4-5.0-H_1x04_P5.00mm_Horizontal -> TerminalBlock_Phoenix:TerminalBlock_Phoenix_PT-1,5-4-3.5-H_1x04_P3.50mm_Horizontal
- K1: footprint Relay_THT:Relay_SPDT_SANYOU_SRD_Series_Form_C -> Display_Segmented:SRA
- SW1, SW2, SW3: footprint Button_Switch_THT:SW_PUSH_6mm_H5mm -> Button_Switch_THT:SW_PUSH_6mm
Connections:
- net A: now also U4.11 (a)
- net B: now also U4.7 (b)
- net C: now also U4.4 (c)
- net D: now also U4.2 (d)
- net DIGIT_1: now also U4.12 (CC1)
- net DIGIT_2: now also U4.9 (CC2)
- net DIGIT_3: now also U4.8 (CC3)
- net DP: now also U4.3 (DPX)
- net E: now also U4.1 (e)
- net F: now also U4.10 (f)
- net G: now also U4.5 (g)
- no-connect marks 2 -> 5
Other:
- note added: "0.28 inch 3-Digit 7-segment LED Display Common Cathode : - 2381AS"
- note removed: "0.28 inch 3-Digit 7-segment LED Display Common Anode : - 2381AS - HS320281K"

Commit message: layout
Connections:
- net +12V: now also K1.2; no longer K1.5
- net at D2.2 (A), Q1.3 (C), R4.2: now also K1.5; no longer K1.2
Other:
- moved on the sheet: K1
Changed lines of the file:
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@@
 	)
 	(no_connect
-		(at 33.02 74.93)
+		(at 33.02 90.17)
 	)
 	(no_connect
@@
 	(wire
 		(pts
-			(xy 30.48 91.44) (xy 30.48 90.17)
+			(xy 30.48 73.66) (xy 30.48 74.93)
 		)
 		(stroke
@@
 	(wire
 		(pts
-			(xy 25.4 73.66) (xy 27.94 73.66)
+			(xy 25.4 91.44) (xy 27.94 91.44)
 		)
 		(stroke
@@
 	(wire
 		(pts
-			(xy 27.94 91.44) (xy 30.48 91.44)
+			(xy 27.94 73.66) (xy 30.48 73.66)
 		)
 		(stroke
@@
 	(wire
 		(pts
-			(xy 27.94 73.66) (xy 27.94 74.93)
+			(xy 27.94 91.44) (xy 27.94 90.17)
 		)
 		(stroke
@@
 	(global_label "K1"
 		(shape input)
-		(at 27.94 91.44 180)
+		(at 27.94 73.66 180)
 		(fields_autoplaced yes)
 		(effects
@@
 		)
 		(property "Intersheetrefs" "${INTERSHEET_REFS}"
-			(at 22.3802 91.44 0)
+			(at 22.3802 73.66 0)
 			(hide yes)
 			(show_name no)
@@
 	(global_label "K0"
 		(shape input)
-		(at 25.4 73.66 180)
+		(at 25.4 91.44 180)
 		(fields_autoplaced yes)
 		(effects
@@
 		)
 		(property "Intersheetrefs" "${INTERSHEET_REFS}"
-			(at 19.8402 73.66 0)
+			(at 19.8402 91.44 0)
 			(hide yes)
 			(show_name no)
@@
 	(symbol
 		(lib_id "Relay:SANYOU_SRD_Form_C")
-		(at 35.56 82.55 0)
-		(mirror y)
+		(at 35.56 82.55 180)
 		(unit 1)
 		(body_style 1)
@@
 		(dnp no)
 		(property "Reference" "K1"
-			(at 46.482 81.3816 0)
+			(at 46.482 83.7184 0)
 			(show_name no)
 			(do_not_autoplace no)
@@
 		)
 		(property "Value" "SRA-12VDC-AL"
-			(at 46.482 83.693 0)
+			(at 46.482 81.407 0)
 			(show_name no)
 			(do_not_autoplace no)
@@
 		)
 		(property "Footprint" "Display_Segmented:SRA"
-			(at 24.13 83.82 0)
+			(at 24.13 81.28 0)
 			(hide yes)
 			(show_name no)
